Commit message: Add Gazebo Sim (Fortress) support: gz_ros2_control, CHOMP pipeline, gripper controller

File: franka_description/robots/common/hand.xacro (robot description, xacro)
@@ -2,5 +2,7 @@
 <robot xmlns:xacro="http://www.ros.org/wiki/xacro" name="hand">
   <!-- safety_distance: Minimum safety distance in [m] by which the collision volumes are expanded and which is enforced during robot motions -->
-  <xacro:macro name="hand" params="connected_to:='' ns:='' rpy:='0 0 0' xyz:='0 0 0' safety_distance:=0">
+  <!-- add_inertials: see panda_arm.xacro - same gate, off by default to keep MuJoCo/real-hardware
+       output unchanged; Gazebo call site sets this true. -->
+  <xacro:macro name="hand" params="connected_to:='' ns:='' rpy:='0 0 0' xyz:='0 0 0' safety_distance:=0 add_inertials:=false">
     <xacro:unless value="${connected_to == ''}">
       <joint name="${ns}_hand_joint" type="fixed">
@@ -11,4 +13,11 @@
     </xacro:unless>
     <link name="${ns}_hand">
+      <xacro:if value="${add_inertials}">
+        <inertial>
+          <origin rpy="0 0 0" xyz="0 0 0.04"/>
+          <mass value="0.81"/>
+          <inertia ixx="0.1" ixy="0" ixz="0" iyy="0.1" iyz="0" izz="0.1"/>
+        </inertial>
+      </xacro:if>
       <visual>
         <geometry>
@@ -54,4 +63,8 @@
     </link>
     <!-- Define the hand_tcp frame -->
+    <!-- No inertial here even when add_inertials is true: this is a fixed reference
+         frame with no visual/collision. It's rigidly attached to ${ns}_hand via a
+         fixed joint, so SDF lumps it into the parent link automatically - giving
+         it a fake mass would double-count the hand's inertia. -->
     <link name="${ns}_hand_tcp"/>
     <joint name="${ns}_hand_tcp_joint" type="fixed">
@@ -61,4 +74,11 @@
     </joint>
     <link name="${ns}_leftfinger">
+      <xacro:if value="${add_inertials}">
+        <inertial>
+          <origin rpy="0 0 0" xyz="0 0.01 0.02"/>
+          <mass value="0.1"/>
+          <inertia ixx="0.1" ixy="0" ixz="0" iyy="0.1" iyz="0" izz="0.1"/>
+        </inertial>
+      </xacro:if>
       <visual>
         <geometry>
@@ -96,4 +116,11 @@
     </link>
     <link name="${ns}_rightfinger">
+      <xacro:if value="${add_inertials}">
+        <inertial>
+          <origin rpy="0 0 0" xyz="0 -0.01 0.02"/>
+          <mass value="0.1"/>
+          <inertia ixx="0.1" ixy="0" ixz="0" iyy="0.1" iyz="0" izz="0.1"/>
+        </inertial>
+      </xacro:if>
       <visual>
         <origin xyz="0 0 0" rpy="0 0 ${pi}"/>
@@ -146,4 +173,13 @@
       <mimic joint="${ns}_finger_joint1"/>
     </joint>
+    <gazebo reference="${ns}_hand">
+      <selfCollide>false</selfCollide>
+    </gazebo>
+    <gazebo reference="${ns}_leftfinger">
+      <selfCollide>false</selfCollide>
+    </gazebo>
+    <gazebo reference="${ns}_rightfinger">
+      <selfCollide>false</selfCollide>
+</gazebo>
   </xacro:macro>
 </robot>

File: franka_description/robots/common/panda_arm.xacro (robot description, xacro)
@@ -3,5 +3,9 @@
   <!-- safety_distance: Minimum safety distance in [m] by which the collision volumes are expanded and which is enforced during robot motions -->
   <!-- arm_id: Namespace of the panda arm. Serves to differentiate between arms in case of multiple instances. -->
-  <xacro:macro name="panda_arm" params="arm_id:='panda' description_pkg:='franka_description' connected_to:='' xyz:='0 0 0' rpy:='0 0 0' safety_distance:=0">
+  <!-- add_inertials: Whether to emit <inertial> blocks. Real hardware and MuJoCo sim don't need
+       this (mass/inertia comes from elsewhere), but Gazebo's urdf2sdf converter requires every
+       link to have one or it silently drops the whole model. Defaults to false to keep the
+       MuJoCo/real-hardware xacro path byte-for-byte unchanged. -->
+  <xacro:macro name="panda_arm" params="arm_id:='panda' description_pkg:='franka_description' connected_to:='' xyz:='0 0 0' rpy:='0 0 0' safety_distance:=0 add_inertials:=false">
     <xacro:unless value="${not connected_to}">
       <joint name="${arm_id}_joint_${connected_to}" type="fixed">
@@ -12,4 +16,11 @@
     </xacro:unless>
     <link name="${arm_id}_link0">
+      <xacro:if value="${add_inertials}">
+        <inertial>
+          <origin rpy="0 0 0" xyz="0 0 0.05"/>
+          <mass value="2.9"/>
+          <inertia ixx="0.1" ixy="0" ixz="0" iyy="0.1" iyz="0" izz="0.1"/>
+        </inertial>
+      </xacro:if>
       <visual>
         <geometry>
@@ -37,4 +48,11 @@
     </link>
     <link name="${arm_id}_link1">
+      <xacro:if value="${add_inertials}">
+        <inertial>
+          <origin rpy="0 0 0" xyz="0 -0.04 -0.05"/>
+          <mass value="2.7"/>
+          <inertia ixx="0.1" ixy="0" ixz="0" iyy="0.1" iyz="0" izz="0.1"/>
+        </inertial>
+      </xacro:if>
       <visual>
         <geometry>
@@ -70,4 +88,11 @@
     </joint>
     <link name="${arm_id}_link2">
+      <xacro:if value="${add_inertials}">
+        <inertial>
+          <origin rpy="0 0 0" xyz="0 -0.04 0.06"/>
+          <mass value="2.73"/>
+          <inertia ixx="0.1" ixy="0" ixz="0" iyy="0.1" iyz="0" izz="0.1"/>
+        </inertial>
+      </xacro:if>
       <visual>
         <geometry>
@@ -103,4 +128,11 @@
     </joint>
     <link name="${arm_id}_link3">
+      <xacro:if value="${add_inertials}">
+        <inertial>
+          <origin rpy="0 0 0" xyz="0.01 0.01 -0.05"/>
+          <mass value="2.04"/>
+          <inertia ixx="0.1" ixy="0" ixz="0" iyy="0.1" iyz="0" izz="0.1"/>
+        </inertial>
+      </xacro:if>
       <visual>
         <geometry>
@@ -136,4 +168,11 @@
     </joint>
     <link name="${arm_id}_link4">
+      <xacro:if value="${add_inertials}">
+        <inertial>
+          <origin rpy="0 0 0" xyz="-0.03 0.03 0.02"/>
+          <mass value="2.08"/>
+          <inertia ixx="0.1" ixy="0" ixz="0" iyy="0.1" iyz="0" izz="0.1"/>
+        </inertial>
+      </xacro:if>
       <visual>
         <geometry>
@@ -169,4 +208,11 @@
     </joint>
     <link name="${arm_id}_link5">
+      <xacro:if value="${add_inertials}">
+        <inertial>
+          <origin rpy="0 0 0" xyz="0 0.04 -0.12"/>
+          <mass value="3.0"/>
+          <inertia ixx="0.1" ixy="0" ixz="0" iyy="0.1" iyz="0" izz="0.1"/>
+        </inertial>
+      </xacro:if>
       <visual>
         <geometry>
@@ -220,4 +266,11 @@
     </joint>
     <link name="${arm_id}_link6">
+      <xacro:if value="${add_inertials}">
+        <inertial>
+          <origin rpy="0 0 0" xyz="0.04 0 0"/>
+          <mass value="1.3"/>
+          <inertia ixx="0.1" ixy="0" ixz="0" iyy="0.1" iyz="0" izz="0.1"/>
+        </inertial>
+      </xacro:if>
       <visual>
         <geometry>
@@ -253,4 +306,11 @@
     </joint>
     <link name="${arm_id}_link7">
+      <xacro:if value="${add_inertials}">
+        <inertial>
+          <origin rpy="0 0 0" xyz="0 0 0.08"/>
+          <mass value="0.2"/>
+          <inertia ixx="0.1" ixy="0" ixz="0" iyy="0.1" iyz="0" izz="0.1"/>
+        </inertial>
+      </xacro:if>
       <visual>
         <geometry>
@@ -286,4 +346,11 @@
     </joint>
     <link name="${arm_id}_link8">
+      <xacro:if value="${add_inertials}">
+        <inertial>
+          <origin rpy="0 0 0" xyz="0 0 0"/>
+          <mass value="0.01"/>
+          <inertia ixx="0.001" ixy="0" ixz="0" iyy="0.001" iyz="0" izz="0.001"/>
+        </inertial>
+      </xacro:if>
       <collision>
         <origin xyz="0.0424 0.0424 -0.0250" rpy="${pi} ${pi/2} ${pi/2}"/>
